File: pcb/aquarius-hub-hw.kicad_sch (KiCad schematic)
At the start: 0 parts

Commit message: Adjusting for consistency
Other:
- title: Hub Hardware -> Aquarius Hub
Changed lines of the file:
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@@
 	(paper "A4")
 	(title_block
-		(title "Hub Hardware")
+		(title "Aquarius Hub")
 		(date "<<release-date>>")
 		(rev "<<tag>>")
